Commit message: fix(model): restore provisional G1 model truth
- amend the schema for provisional actuators, nullable photos, armature, and NR verification

- preserve source armature values through ingestion and MJCF emission

- emit primitive URDF collisions with MJCF-native dimension conversions

- regenerate model and simulator artifacts after restoring truthful provisional fields

File: model/generated/robot.urdf (robot description, URDF)
Before this commit: robot unitree_g1, 30 links, 29 joints
Links:
- link left_ankle_roll_link: geometry collision mesh filename=../source/menagerie/unitree_g1/assets/left_ankle_roll_link; collision sphere radius=0.005
- link left_shoulder_pitch_link: geometry collision cylinder length=0.05 radius=0.03; collision mesh filename=../source/menagerie/unitree_g1/assets/left_shoulder_pitch_l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
- link left_shoulder_roll_link: geometry collision cylinder length=0.03 radius=0.03; collision mesh filename=../source/menagerie/unitree_g1/assets/left_shoulder_roll_li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
- link right_ankle_roll_link: geometry collision mesh filename=../source/menagerie/unitree_g1/assets/right_ankle_roll_link; collision sphere radius=0.005
- link right_shoulder_pitch_link: geometry collision cylinder length=0.05 radius=0.03; collision mesh filename=../source/menagerie/unitree_g1/assets/right_shoulder_pitch_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
- link right_shoulder_roll_link: geometry collision cylinder length=0.03 radius=0.03; collision mesh filename=../source/menagerie/unitree_g1/assets/right_shoulder_roll_l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

Commit message: refactor(urdf)!: support absolute mesh file URIs
- update URDF emission to accept absolute mesh file URIs
- preserve relative asset paths for existing model setups
- simplify downstream mesh loading for the MuJoCo transport stack

BREAKING CHANGE: mesh emission now expects absolute file URIs for asset paths, and consumers must adapt to the new URI handling.

File: model/generated/robot.urdf (robot description, URDF)
Before this commit: robot unitree_g1, 30 links, 29 joints
Links:
- link left_ankle_pitch_link: geometry collision mesh filename=file:///ws/model/source/menagerie/unitree_g1/assets/left_an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; visual mesh filename=file:///ws/model/source/menagerie/unitree_g1/assets/left_an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
- link left_ankle_roll_link: geometry collision mesh filename=file:///ws/model/source/menagerie/unitree_g1/assets/left_an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; collision sphere radius=0.005
- link left_elbow_link: geometry collision mesh filename=file:///ws/model/source/menagerie/unitree_g1/assets/left_el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; visual mesh filename=file:///ws/model/source/menagerie/unitree_g1/assets/left_el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
- link left_hip_pitch_link: geometry collision mesh filename=file:///ws/model/source/menagerie/unitree_g1/assets/left_hi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; visual mesh filename=file:///ws/model/source/menagerie/unitree_g1/assets/left_hi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
- link left_hip_roll_link: geometry collision mesh filename=file:///ws/model/source/menagerie/unitree_g1/assets/left_hi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; visual mesh filename=file:///ws/model/source/menagerie/unitree_g1/assets/left_hi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
- link left_hip_yaw_link: geometry collision mesh filename=file:///ws/model/source/menagerie/unitree_g1/assets/left_hi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; visual mesh filename=file:///ws/model/source/menagerie/unitree_g1/assets/left_hi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
- link left_knee_link: geometry collision mesh filename=file:///ws/model/source/menagerie/unitree_g1/assets/left_kn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; visual mesh filename=file:///ws/model/source/menagerie/unitree_g1/assets/left_kn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
- link left_shoulder_pitch_link: geometry collision cylinder length=0.05 radius=0.03; collision mesh filename=file:///ws/model/source/menagerie/unitree_g1/assets/left_sh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
- link left_shoulder_roll_link: geometry collision cylinder length=0.03 radius=0.03; collision mesh filename=file:///ws/model/source/menagerie/unitree_g1/assets/left_sh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
- link left_shoulder_yaw_link: geometry collision mesh filename=file:///ws/model/source/menagerie/unitree_g1/assets/left_sh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; visual mesh filename=file:///ws/model/source/menagerie/unitree_g1/assets/left_sh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
- link left_wrist_pitch_link: geometry collision mesh filename=file:///ws/model/source/menagerie/unitree_g1/assets/left_wr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; visual mesh filename=file:///ws/model/source/menagerie/unitree_g1/assets/left_wr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
- link left_wrist_roll_link: geometry collision mesh filename=file:///ws/model/source/menagerie/unitree_g1/assets/left_wr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; visual mesh filename=file:///ws/model/source/menagerie/unitree_g1/assets/left_wr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
- link left_wrist_yaw_link: geometry collision mesh filename=file:///ws/model/source/menagerie/unitree_g1/assets/left_wr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; visual mesh filename=file:///ws/model/source/menagerie/unitree_g1/assets/left_wr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
- link pelvis: geometry collision mesh filename=file:///ws/model/source/menagerie/unitree_g1/assets/pelvis_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; visual mesh filename=file:///ws/model/source/menagerie/unitree_g1/assets/pelvis_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
- link right_ankle_pitch_link: geometry collision mesh filename=file:///ws/model/source/menagerie/unitree_g1/assets/right_a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; visual mesh filename=file:///ws/model/source/menagerie/unitree_g1/assets/right_a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
- link right_ankle_roll_link: geometry collision mesh filename=file:///ws/model/source/menagerie/unitree_g1/assets/right_a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; collision sphere radius=0.005
- link right_elbow_link: geometry collision mesh filename=file:///ws/model/source/menagerie/unitree_g1/assets/right_e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; visual mesh filename=file:///ws/model/source/menagerie/unitree_g1/assets/right_e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
- link right_hip_pitch_link: geometry collision mesh filename=file:///ws/model/source/menagerie/unitree_g1/assets/right_h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; visual mesh filename=file:///ws/model/source/menagerie/unitree_g1/assets/right_h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
- link right_hip_roll_link: geometry collision mesh filename=file:///ws/model/source/menagerie/unitree_g1/assets/right_h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; visual mesh filename=file:///ws/model/source/menagerie/unitree_g1/assets/right_h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
- link right_hip_yaw_link: geometry collision mesh filename=file:///ws/model/source/menagerie/unitree_g1/assets/right_h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; visual mesh filename=file:///ws/model/source/menagerie/unitree_g1/assets/right_h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
- link right_knee_link: geometry collision mesh filename=file:///ws/model/source/menagerie/unitree_g1/assets/right_k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; visual mesh filename=file:///ws/model/source/menagerie/unitree_g1/assets/right_k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
- link right_shoulder_pitch_link: geometry collision cylinder length=0.05 radius=0.03; collision mesh filename=file:///ws/model/source/menagerie/unitree_g1/assets/right_s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
- link right_shoulder_roll_link: geometry collision cylinder length=0.03 radius=0.03; collision mesh filename=file:///ws/model/source/menagerie/unitree_g1/assets/right_s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
- link right_shoulder_yaw_link: geometry collision mesh filename=file:///ws/model/source/menagerie/unitree_g1/assets/right_s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; visual mesh filename=file:///ws/model/source/menagerie/unitree_g1/assets/right_s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
- link right_wrist_pitch_link: geometry collision mesh filename=file:///ws/model/source/menagerie/unitree_g1/assets/right_w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; visual mesh filename=file:///ws/model/source/menagerie/unitree_g1/assets/right_w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
- link right_wrist_roll_link: geometry collision mesh filename=file:///ws/model/source/menagerie/unitree_g1/assets/right_w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; visual mesh filename=file:///ws/model/source/menagerie/unitree_g1/assets/right_w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
- link right_wrist_yaw_link: geometry collision mesh filename=file:///ws/model/source/menagerie/unitree_g1/assets/right_w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; visual mesh filename=file:///ws/model/source/menagerie/unitree_g1/assets/right_w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
- link torso_link: geometry collision mesh filename=file:///ws/model/source/menagerie/unitree_g1/assets/torso_l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; visual mesh filename=file:///ws/model/source/menagerie/unitree_g1/assets/torso_l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
- link waist_roll_link: geometry collision mesh filename=file:///ws/model/source/menagerie/unitree_g1/assets/waist_r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; visual mesh filename=file:///ws/model/source/menagerie/unitree_g1/assets/waist_r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
- link waist_yaw_link: geometry collision mesh filename=file:///ws/model/source/menagerie/unitree_g1/assets/waist_y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; visual mesh filename=file:///ws/model/source/menagerie/unitree_g1/assets/waist_y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
